Commit message: OpenCR implements the new interface UsbDevice
Removed all references to wheels, imu, battery

File: open_manipulator_description/ros2_control/open_manipulator_system.ros2_control.xacro (robot description, xacro)
@@ -6,5 +6,5 @@
 -->
 <robot xmlns:xacro="http://www.ros.org/wiki/xacro">
-  <xacro:macro name="open_manipulator_system" params="name prefix use_sim:=^|false use_fake_hardware:=^|false fake_sensor_commands:=^|false">
+  <xacro:macro name="open_manipulator_system" params="name prefix use_sim:=^|false use_fake_hardware:=^|false fake_sensor_commands:=^|false usb_port baud_rate">
     <ros2_control name="${name}" type="system">
       <xacro:if value="$(arg use_sim)">
@@ -23,6 +23,6 @@
             <plugin>open_manipulator_hardware/OpenManipulatorManipulationSystemHardware</plugin>
             <param name="opencr_id">200</param>
-            <param name="opencr_usb_port">/dev/ttyACM0</param>
-            <param name="opencr_baud_rate">1000000</param>
+            <param name="opencr_usb_port">${usb_port}</param>
+            <param name="opencr_baud_rate">${baud_rate}</param>
             <param name="dxl_joints_profile_acceleration">100</param>
             <param name="dxl_joints_profile_velocity">500</param>

File: open_manipulator_description/urdf/open_manipulator.urdf.xacro (robot description, xacro)
@@ -6,4 +6,6 @@
   <xacro:arg name="use_fake_hardware" default="false" />
   <xacro:arg name="fake_sensor_commands" default="false" />
+  <xacro:arg name="usb_port" default="/dev/ttyUSB0" />
+  <xacro:arg name="baud_rate" default="1000000" />
   <!-- Import materials macro -->
   <xacro:include filename="$(find open_manipulator_description)/gazebo/materials.xacro" />
@@ -19,5 +21,8 @@
     name="OpenManipulatorManipulationSystem" prefix="$(arg prefix)" use_sim="$(arg use_sim)"
     use_fake_hardware="$(arg use_fake_hardware)"
-    fake_sensor_commands="$(arg fake_sensor_commands)"/>
+    fake_sensor_commands="$(arg fake_sensor_commands)"
+    usb_port="$(arg usb_port)"
+    baud_rate="$(arg baud_rate)"
+    />
   <gazebo>
     <plugin name="gazebo_ros2_control" filename="libgazebo_ros2_control.so">

Commit message: Added U2D2 as implementation of UsbDevice
Building, but errors at runtime that need to be fixed

File: open_manipulator_description/ros2_control/open_manipulator_system.ros2_control.xacro (robot description, xacro)
@@ -6,5 +6,5 @@
 -->
 <robot xmlns:xacro="http://www.ros.org/wiki/xacro">
-  <xacro:macro name="open_manipulator_system" params="name prefix use_sim:=^|false use_fake_hardware:=^|false fake_sensor_commands:=^|false usb_port baud_rate">
+  <xacro:macro name="open_manipulator_system" params="name prefix use_sim:=^|false use_fake_hardware:=^|false fake_sensor_commands:=^|false usb_port usb_device baud_rate">
     <ros2_control name="${name}" type="system">
       <xacro:if value="$(arg use_sim)">
@@ -22,7 +22,8 @@
           <xacro:unless value="${use_fake_hardware}">
             <plugin>open_manipulator_hardware/OpenManipulatorManipulationSystemHardware</plugin>
-            <param name="opencr_id">200</param>
-            <param name="opencr_usb_port">${usb_port}</param>
-            <param name="opencr_baud_rate">${baud_rate}</param>
+            <param name="manipulator_id">200</param>
+            <param name="manipulator_usb_port">${usb_port}</param>
+            <param name="manipulator_usb_device">${usb_device}</param>
+            <param name="manipulator_baud_rate">${baud_rate}</param>
             <param name="dxl_joints_profile_acceleration">100</param>
             <param name="dxl_joints_profile_velocity">500</param>

File: open_manipulator_description/urdf/open_manipulator.urdf.xacro (robot description, xacro)
@@ -7,4 +7,5 @@
   <xacro:arg name="fake_sensor_commands" default="false" />
   <xacro:arg name="usb_port" default="/dev/ttyUSB0" />
+  <xacro:arg name="usb_device" default="u2d2" />
   <xacro:arg name="baud_rate" default="1000000" />
   <!-- Import materials macro -->
@@ -23,4 +24,5 @@
     fake_sensor_commands="$(arg fake_sensor_commands)"
     usb_port="$(arg usb_port)"
+    usb_device="$(arg usb_device)"
     baud_rate="$(arg baud_rate)"
     />
